File: Trans1/trans1.sch (EAGLE design)
At the start: 21 parts, among them Q1 MOSFET-NCHANNELBSS138, Q2 BC817-16LT1SMD, U1 DRA818V

Commit message: Version 1.03
Added third pole to RF filter, adjusted pad size on DRA module.
Parts:
- removed SV1: (no value), con-lstb:MA03-1
- added C5: .1uF, resistor:C-USC0805
- added J2: (no value), con-lstb:MA03-1
- added L3: 1µH, custom-ds:INDUCTOR
- C1, C4: value (none) -> 20pF
- C2, C3: value (none) -> 36pF
- D1: value (none) -> 1N4148
- L1, L2: value (none) -> 1µH; device SparkFun-Passives:INDUCTOR0805 -> custom-ds:INDUCTOR
- Q1: value MOSFET-NCHANNELBSS138 -> BC817-16LT1SMD; device SparkFun-DiscreteSemi:MOSFET-NCHANNELBSS138 -> transistor-npn:BC817-16LT1SMD; DIGIKEY (none) -> MMBT2222AFSCT-ND
- Q2: value BC817-16LT1SMD -> MOSFET-NCHANNELBSS138; device transistor-npn:BC817-16LT1SMD -> SparkFun-DiscreteSemi:MOSFET-NCHANNELBSS138; DIGIKEY MMBT2222AFSCT-ND -> (none)
- R1, R2, R5, R6: value (none) -> 10k
- R3, R4: value (none) -> 1k
- R7: value (none) -> 100k
- U1: device DRA818V:DRA818V -> custom-ds:DRA818V
- renumbered SV3 to J1
Connections:
- removed net N$8: C1.1, L1.1, SV1.2
- new net N$10: C1.1, J2.2, L1.1
- new net N$7: C3.1, L2.2, L3.1
- net +5V: now also R5.2; no longer R7.2
- net GND: now also C5.2, J2.1, J2.3, Q1.E, R1.1, R7.1; no longer Q2.E, R2.1, R5.1, SV1.1, SV1.3
- net N$1: now also Q1.C, R3.1; no longer Q2.C, R7.1
- net N$2: now also R1.2; no longer R2.2
- net N$3: now also R6.2, R7.2; no longer R4.2, R5.2
- net N$4: now also Q2.S, R2.1; no longer Q1.S, R1.1
- net N$5: now also Q1.B, R4.2; no longer Q2.B, R6.2
- net N$6: now also C4.1, L3.2; no longer C3.1, L2.2
- net PTT: now also R4.1; no longer R6.1
- net RX_DATA: now also Q2.D, R5.1; no longer Q1.D, R3.1
- net TX_DATA: now also R6.1; no longer R4.1
- net V+: now also C5.1, Q2.G, R2.2; no longer C4.1, Q1.G, R1.2
Other:
- moved on the sheet: C1, C2, C3, C4, R1, R2, R3, R4, R5, R6, R7

Commit message: Updating part values
Parts:
- C1, C4: DIGIKEY (none) -> ‎712-1381-1-ND‎
- C2, C3: DIGIKEY (none) -> 478-10473-1-ND
- L1, L3: value 1µH -> 56nH; DIGIKEY (none) -> 535-11570-1-ND
- L2: value 1µH -> 68nH; DIGIKEY (none) -> ‎535-11572-1-ND‎
Changed lines of the file:
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@@
 <part name="R5" library="resistor" deviceset="R-US_" device="R0805" value="10k"/>
 <part name="R2" library="resistor" deviceset="R-US_" device="R0805" value="10k"/>
-<part name="C3" library="resistor" deviceset="C-US" device="C0805" value="36pF"/>
-<part name="C4" library="resistor" deviceset="C-US" device="C0805" value="20pF"/>
-<part name="C2" library="resistor" deviceset="C-US" device="C0805" value="36pF"/>
+<part name="C3" library="resistor" deviceset="C-US" device="C0805" value="36pF">
+<attribute name="DIGIKEY" value="478-10473-1-ND"/>
+</part>
+<part name="C4" library="resistor" deviceset="C-US" device="C0805" value="20pF">
+<attribute name="DIGIKEY" value="‎712-1381-1-ND‎"/>
+</part>
+<part name="C2" library="resistor" deviceset="C-US" device="C0805" value="36pF">
+<attribute name="DIGIKEY" value="478-10473-1-ND"/>
+</part>
 <part name="C5" library="resistor" deviceset="C-US" device="C0805" value=".1uF"/>
 <part name="Q2" library="SparkFun-DiscreteSemi" deviceset="MOSFET-NCHANNEL" device="BSS138"/>
 <part name="JP1" library="SparkFun-Connectors" deviceset="M01" device="PTH"/>
 <part name="JP2" library="SparkFun-Connectors" deviceset="M01" device="PTH"/>
-<part name="L2" library="custom-ds" deviceset="INDUCTOR" device="" value="1µH"/>
-<part name="L3" library="custom-ds" deviceset="INDUCTOR" device="" value="1µH"/>
+<part name="L2" library="custom-ds" deviceset="INDUCTOR" device="" value="68nH">
+<attribute name="DIGIKEY" value="‎535-11572-1-ND‎"/>
+</part>
+<part name="L3" library="custom-ds" deviceset="INDUCTOR" device="" value="56nH">
+<attribute name="DIGIKEY" value="535-11570-1-ND"/>
+</part>
 <part name="R1" library="resistor" deviceset="R-US_" device="R0805" value="10k"/>
 <part name="GND6" library="supply1" deviceset="GND" device=""/>
@@
 <part name="R3" library="resistor" deviceset="R-US_" device="R0805" value="1k"/>
 <part name="P+3" library="supply1" deviceset="+5V" device=""/>
-<part name="L1" library="custom-ds" deviceset="INDUCTOR" device="" value="1µH"/>
-<part name="C1" library="resistor" deviceset="C-US" device="C0805" value="20pF"/>
+<part name="L1" library="custom-ds" deviceset="INDUCTOR" device="" value="56nH">
+<attribute name="DIGIKEY" value="535-11570-1-ND"/>
+</part>
+<part name="C1" library="resistor" deviceset="C-US" device="C0805" value="20pF">
+<attribute name="DIGIKEY" value="‎712-1381-1-ND‎"/>
+</part>
 </parts>
 <sheets>
@@
 <instance part="R5" gate="G$1" x="149.86" y="134.62" rot="R90"/>
 <instance part="R2" gate="G$1" x="124.46" y="134.62" rot="R90"/>
-<instance part="C3" gate="G$1" x="43.18" y="73.66"/>
-<instance part="C4" gate="G$1" x="58.42" y="73.66"/>
-<instance part="C2" gate="G$1" x="27.94" y="73.66"/>
+<instance part="C3" gate="G$1" x="43.18" y="73.66">
+<attribute name="DIGIKEY" x="43.18" y="73.66" size="1.778" layer="96" display="off"/>
+</instance>
+<instance part="C4" gate="G$1" x="58.42" y="73.66">
+<attribute name="DIGIKEY" x="58.42" y="73.66" size="1.778" layer="96" display="off"/>
+</instance>
+<instance part="C2" gate="G$1" x="27.94" y="73.66">
+<attribute name="DIGIKEY" x="27.94" y="73.66" size="1.778" layer="96" display="off"/>
+</instance>
 <instance part="C5" gate="G$1" x="93.98" y="38.1"/>
 <instance part="Q2" gate="G$1" x="137.16" y="124.46" rot="R270"/>
 <instance part="JP1" gate="G$1" x="177.8" y="81.28"/>
 <instance part="JP2" gate="G$1" x="177.8" y="68.58"/>
-<instance part="L2" gate="G$1" x="35.56" y="81.28" rot="R90"/>
-<instance part="L3" gate="G$1" x="50.8" y="81.28" rot="R90"/>
+<instance part="L2" gate="G$1" x="35.56" y="81.28" rot="R90">
+<attribute name="DIGIKEY" x="35.56" y="81.28" size="1.778" layer="96" rot="R90" display="off"/>
+</instance>
+<instance part="L3" gate="G$1" x="50.8" y="81.28" rot="R90">
+<attribute name="DIGIKEY" x="50.8" y="81.28" size="1.778" layer="96" rot="R90" display="off"/>
+</instance>
 <instance part="R1" gate="G$1" x="109.22" y="76.2" rot="R90"/>
 <instance part="GND6" gate="1" x="170.18" y="30.48"/>
@@
 <instance part="R3" gate="G$1" x="127" y="101.6" rot="R90"/>
 <instance part="P+3" gate="1" x="127" y="111.76"/>
-<instance part="L1" gate="G$1" x="20.32" y="81.28" rot="R90"/>
-<instance part="C1" gate="G$1" x="12.7" y="73.66"/>
+<instance part="L1" gate="G$1" x="20.32" y="81.28" rot="R90">
+<attribute name="DIGIKEY" x="20.32" y="81.28" size="1.778" layer="96" rot="R90" display="off"/>
+</instance>
+<instance part="C1" gate="G$1" x="12.7" y="73.66">
+<attribute name="DIGIKEY" x="12.7" y="73.66" size="1.778" layer="96" display="off"/>
+</instance>
 </instances>
 <busses>
